Commit message: tomato with collision

File: urdf_robot/tomato_plant.urdf (robot description, URDF)
Before this commit: robot tomato, 5 links, 4 joints
Links:
- link tomato: geometry collision mesh filename=tomato/10208_TomatoBeefSteak_v1.obj scale=0.01 0.01 0.01; visual mesh filename=tomato/10208_TomatoBeefSteak_v1.obj scale=0.01 0.01 0.01
- link tomato2: geometry collision mesh filename=tomato/10208_TomatoBeefSteak_v1.obj scale=0.006 0.006 0.006; visual mesh filename=tomato/10208_TomatoBeefSteak_v1.obj scale=0.006 0.006 0.006
- link tomato3: geometry collision mesh filename=tomato/10208_TomatoBeefSteak_v1.obj scale=0.008 0.008 0.008; visual mesh filename=tomato/10208_TomatoBeefSteak_v1.obj scale=0.008 0.008 0.008
- link tomato4: geometry collision mesh filename=tomato/10208_TomatoBeefSteak_v1.obj scale=0.005 0.005 0.005; visual mesh filename=tomato/10208_TomatoBeefSteak_v1.obj scale=0.005 0.005 0.005
