Commit message: joint_limits update

File: urdf_robot/inmoov_col.urdf (robot description, URDF)
Before this commit: robot inmoov, 87 links, 86 joints
Joints:
- joint left_bicep: limit lower=0.0 upper=-3.1415926 effort=1000.0 velocity=0.5 -> lower=0.0 upper=-1.5707963 effort=1000.0 velocity=0.5
- joint right_bicep: limit lower=-3.1415926 upper=0.0 effort=1000.0 velocity=0.5 -> lower=-1.5707963 upper=0.0 effort=1000.0 velocity=0.5
