Commit message: jaka obstacle&inmoov remote control

File: urdf/long_cylinder.urdf (robot description, URDF)
Before this commit: robot cylinder, 1 links, 0 joints
Links:
- link cylinder_button: geometry collision mesh filename=meshes/button.dae scale=0.2 0.2 40.0; visual mesh filename=meshes/button.dae scale=0.2 0.2 40.0
